Commit message: replace wheel_stuck_alpha to wheel_stuck_go
Signed-off-by: Autumn60 <harada.akiro@gmail.com>

File: src/description/wheel_stuck_go/wheel_stuck_go_description/urdf/robot.urdf.xacro (robot description, xacro)
@@ -1,5 +1,5 @@
 <?xml version="1.0"?>
 <robot xmlns:xacro="http://ros.org/wiki/xacro">
-  <xacro:property name="robot_info" value="${xacro.load_yaml('$(find wheel_stuck_alpha_description)/config/robot_info.param.yaml')}"/>
+  <xacro:property name="robot_info" value="${xacro.load_yaml('$(find wheel_stuck_go_description)/config/robot_info.param.yaml')}"/>
   <link name="base_link"/>
 </robot>

File: src/description/wheel_stuck_go/wheel_stuck_go_sensor_kit_description/urdf/sensor_kit.urdf.xacro (robot description, xacro)
@@ -1,5 +1,5 @@
 <?xml version="1.0"?>
 <robot xmlns:xacro="http://ros.org/wiki/xacro">
-  <xacro:property name="sensors_calibration" value="${xacro.load_yaml('$(find wheel_stuck_alpha_sensor_kit_description)/config/sensors_calibration.param.yaml')}"/>
+  <xacro:property name="sensors_calibration" value="${xacro.load_yaml('$(find wheel_stuck_go_sensor_kit_description)/config/sensors_calibration.param.yaml')}"/>
   <link name="velodyne_base_link"/>
   <joint name="velodyne_base_joint" type="fixed">
