Commit message: create xacro macro for sensors
Signed-off-by: Autumn60 <harada.akiro@gmail.com>

File: src/description/fourth_robot/fourth_robot_sensor_kit_description/urdf/sensor_kit.urdf.xacro (robot description, xacro)
@@ -2,35 +2,19 @@
 <robot xmlns:xacro="http://ros.org/wiki/xacro">
   <xacro:property name="sensors_calibration" value="${xacro.load_yaml('$(find fourth_robot_sensor_kit_description)/config/sensors_calibration.param.yaml')}"/>
-  <link name="front_lrf_link">
-    <visual>
-      <origin xyz="0 0 0" rpy="0 0 0"/>
-      <geometry>
-        <mesh filename="package://fourth_robot_sensor_kit_description/mesh/front_lrf/front_lrf.dae" scale="1 1 1"/>
-      </geometry>
-    </visual>
-  </link>
-  <joint name="front_lrf_joint" type="fixed">
-    <parent link="base_link"/>
-    <child link="front_lrf_link"/>
+  <xacro:include filename="$(find fourth_robot_sensor_kit_description)/urdf/front_lrf/front_lrf.urdf.xacro"/>
+  <xacro:include filename="$(find fourth_robot_sensor_kit_description)/urdf/rear_lrf/rear_lrf.urdf.xacro"/>
+  <xacro:include filename="$(find fourth_robot_sensor_kit_description)/urdf/gim30/gim30.urdf.xacro"/>
+  <xacro:include filename="$(find fourth_robot_sensor_kit_description)/urdf/gps/gps.urdf.xacro"/>
+  <xacro:front_lrf name="front_lrf" parent="base_link">
     <origin
       xyz="${sensors_calibration['base_link']['front_lrf_link']['x']}
-             ${sensors_calibration['base_link']['front_lrf_link']['y']}
-             ${sensors_calibration['base_link']['front_lrf_link']['z']}"
+              ${sensors_calibration['base_link']['front_lrf_link']['y']}
+              ${sensors_calibration['base_link']['front_lrf_link']['z']}"
       rpy="${sensors_calibration['base_link']['front_lrf_link']['roll']}
-             ${sensors_calibration['base_link']['front_lrf_link']['pitch']}
-            ${sensors_calibration['base_link']['front_lrf_link']['yaw']}"
+              ${sensors_calibration['base_link']['front_lrf_link']['pitch']}
+              ${sensors_calibration['base_link']['front_lrf_link']['yaw']}"
     />
-  </joint>
-  <link name="rear_lrf_link">
-    <visual>
-      <origin xyz="0 0 0" rpy="0 0 0"/>
-      <geometry>
-        <mesh filename="package://fourth_robot_sensor_kit_description/mesh/rear_lrf/rear_lrf.dae" scale="1 1 1"/>
-      </geometry>
-    </visual>
-  </link>
-  <joint name="rear_lrf_joint" type="fixed">
-    <parent link="base_link"/>
-    <child link="rear_lrf_link"/>
+  </xacro:front_lrf>
+  <xacro:rear_lrf name="rear_lrf" parent="base_link">
     <origin
       xyz="${sensors_calibration['base_link']['rear_lrf_link']['x']}
@@ -41,16 +25,6 @@
               ${sensors_calibration['base_link']['rear_lrf_link']['yaw']}"
     />
-  </joint>
-  <link name="gim30_link">
-    <visual>
-      <origin xyz="0 0 0" rpy="0 0 0"/>
-      <geometry>
-        <mesh filename="package://fourth_robot_sensor_kit_description/mesh/gim30/gim30.dae" scale="1 1 1"/>
-      </geometry>
-    </visual>
-  </link>
-  <joint name="gim30_joint" type="fixed">
-    <parent link="base_link"/>
-    <child link="gim30_link"/>
+  </xacro:rear_lrf>
+  <xacro:gim30 name="gim30" parent="base_link">
     <origin
       xyz="${sensors_calibration['base_link']['gim30_link']['x']}
@@ -61,16 +35,6 @@
               ${sensors_calibration['base_link']['gim30_link']['yaw']}"
     />
-  </joint>
-  <link name="gps_link">
-    <visual>
-      <origin xyz="0 0 0" rpy="0 0 0"/>
-      <geometry>
-        <mesh filename="package://fourth_robot_sensor_kit_description/mesh/gps/gps.dae" scale="1 1 1"/>
-      </geometry>
-    </visual>
-  </link>
-  <joint name="gps_joint" type="fixed">
-    <parent link="base_link"/>
-    <child link="gps_link"/>
+  </xacro:gim30>
+  <xacro:gps name="gps" parent="base_link">
     <origin
       xyz="${sensors_calibration['base_link']['gps_link']['x']}
@@ -81,4 +45,4 @@
               ${sensors_calibration['base_link']['gps_link']['yaw']}"
     />
-  </joint>
+  </xacro:gps>
 </robot>
